Commit message: Fix link_r1 mass issue, and del the ee link

File: urdf/astra_description.urdf (robot description, URDF)
Before this commit: robot astra_description, 19 links, 18 joints
Links:
- removed link link_eel
- removed link link_eer
- link base_link: mass 16.662 -> 16.658
- link link_l1: mass 0 -> 0.68712
- link link_l2: mass 0.752093604412347 -> 0.75209
- link link_l3: mass 0.397219077227713 -> 0.39722
- link link_l4: mass 0.0805715795068273 -> 0.080572
- link link_l5: mass 0.0769437691997218 -> 0.076944
- link link_r1: mass 0.687116799139831 -> 0.68712
- link link_r2: mass 0.75209360511139 -> 0.75209
- link link_r3: mass 0.397219076403374 -> 0.39722
- link link_r4: mass 0.0805715790970505 -> 0.080572
- link link_r5: mass 0.076943769270768 -> 0.076944
- link link_r6: mass 0.116566142920341 -> 0.11657
Joints:
- removed joint joint_eel
- removed joint joint_eer

Commit message: Add end effector fixed link

File: urdf/astra_description.urdf (robot description, URDF)
Before this commit: robot astra_description, 17 links, 16 joints
Links:
- added link link_lee
- added link link_ree
Joints:
- added joint joint_lee: type fixed, parent link_l6, child link_lee, origin xyz=0.063 0 0.195 rpy=3.1416 -1.5708 0, axis 0 0 0
- added joint joint_ree: type fixed, parent link_r6, child link_ree, origin xyz=0.063 0 0.195 rpy=1.5708 -1.5708 0, axis 0 0 0

Commit message: Fix end effector wrong rotation

File: urdf/astra_description.urdf (robot description, URDF)
Before this commit: robot astra_description, 19 links, 18 joints
Joints:
- joint joint_lee: axis 0 0 0 -> (none); origin xyz=0.063 0 0.195 rpy=3.1416 -1.5708 0 -> xyz=0.063 0 0.195 rpy=0 -1.5708 0
- joint joint_ree: axis 0 0 0 -> (none); origin xyz=0.063 0 0.195 rpy=1.5708 -1.5708 0 -> xyz=0.063 0 0.195 rpy=0 -1.5708 0

File: urdf/astra_description_rel.urdf (robot description, URDF)
Before this commit: robot astra_description, 19 links, 18 joints
Joints:
- joint joint_lee: origin xyz=0.063 0 0.195 rpy=3.1416 -1.5708 0 -> xyz=0.063 0 0.195 rpy=0 -1.5708 0
- joint joint_ree: axis 0 0 0 -> (none); origin xyz=0.063 0 0.195 rpy=1.5708 -1.5708 0 -> xyz=0.063 0 0.195 rpy=0 -1.5708 0

Commit message: Change new type of lift

File: urdf/astra_description.urdf (robot description, URDF)
Before this commit: robot astra_description, 19 links, 18 joints
Links:
- added link link_head_pan, mass 0.087098; collision mesh filename=package://astra_description/meshes/link_head_pan.STL; visual mesh filename=package://astra_description/meshes/link_head_pan.STL
- added link link_head_tilt, mass 0.032288; collision mesh filename=package://astra_description/meshes/link_head_tilt.STL; visual mesh filename=package://astra_description/meshes/link_head_tilt.STL
- link base_link: mass 16.658 -> 17.285
- link link_l1: mass 0.68712 -> 0.70739
- link link_l4: mass 0.080572 -> 0.087098
- link link_l5: mass 0.076944 -> 0.071465
- link link_l6: mass 0.11657 -> 0.13935
- link link_r1: mass 0.68712 -> 0.70739
- link link_r4: mass 0.080572 -> 0.087098
- link link_r6: mass 0.11657 -> 0.13935
Joints:
- added joint joint_head_pan: type revolute, parent base_link, child link_head_pan, origin xyz=0.05 0 1.429 rpy=-3.1416 0 0, axis 0 0 1, limit lower=-1.57 upper=1.57 effort=0 velocity=0
- added joint joint_head_tilt: type revolute, parent link_head_pan, child link_head_tilt, origin xyz=0 0 0 rpy=1.5708 0 0, axis 0 0 1, limit lower=-3.14 upper=3.14 effort=0 velocity=0
- joint joint_l1: limit lower=0 upper=1 effort=0 velocity=0 -> lower=0 upper=1.2 effort=0 velocity=0; origin xyz=-0.025 0.0755 0.2178 rpy=0 0 1.5708 -> xyz=-0.0405 0.065 0.227 rpy=0 0 1.5708
- joint joint_l2: origin xyz=0.075 0 0 rpy=0 0 -0.18555 -> xyz=0.068 0 0 rpy=0 0 -0.18555
- joint joint_l4: limit lower=-1.57 upper=1.57 effort=0 velocity=0 -> lower=-3.14 upper=3.14 effort=0 velocity=0; origin xyz=0.265 0 -0.079 rpy=3.1416 0 0 -> xyz=0.265 0 -0.087 rpy=3.1416 0 0
- joint joint_l6: origin xyz=0 0 0 rpy=1.5708 0 0 -> xyz=0 0 0 rpy=-1.5708 0 0
- joint joint_l7l: origin xyz=0.063 0 0.195 rpy=1.5708 -1.5708 0 -> xyz=0.078 0 0.195 rpy=1.5708 -1.5708 0
- joint joint_l7r: origin xyz=0.063 0 0.195 rpy=1.5708 -1.5708 0 -> xyz=0.078 0 0.195 rpy=1.5708 -1.5708 0
- joint joint_lee: axis (none) -> 0 0 0
- joint joint_r1: limit lower=0 upper=1 effort=0 velocity=0 -> lower=0 upper=1.2 effort=0 velocity=0; origin xyz=-0.025 -0.0755 0.2178 rpy=0 0 -1.5708 -> xyz=-0.0405 -0.065 0.227 rpy=0 0 -1.5708
- joint joint_r2: origin xyz=0.075 0 0 rpy=0 0 0.18555 -> xyz=0.068 0 0 rpy=0 0 0.18555
- joint joint_r4: limit lower=-1.57 upper=1.57 effort=0 velocity=0 -> lower=-3.14 upper=3.14 effort=0 velocity=0; origin xyz=0.265 0 -0.079 rpy=3.1416 0 0 -> xyz=0.265 0 -0.087 rpy=3.1416 0 0
- joint joint_r7l: origin xyz=0.063 0 0.195 rpy=1.5708 -1.5708 0 -> xyz=0.078 0 0.195 rpy=1.5708 -1.5708 0
- joint joint_r7r: origin xyz=0.063 0 0.195 rpy=1.5708 -1.5708 0 -> xyz=0.078 0 0.195 rpy=1.5708 -1.5708 0

File: urdf/astra_description_rel.urdf (robot description, URDF)
Before this commit: robot astra_description, 19 links, 18 joints
Links:
- added link link_head_pan, mass 0.087098; collision mesh filename=../meshes/link_head_pan.STL; visual mesh filename=../meshes/link_head_pan.STL
- added link link_head_tilt, mass 0.032288; collision mesh filename=../meshes/link_head_tilt.STL; visual mesh filename=../meshes/link_head_tilt.STL
- link base_link: mass 16.658 -> 17.285
- link link_l1: mass 0.68712 -> 0.70739
- link link_l4: mass 0.080572 -> 0.087098
- link link_l5: mass 0.076944 -> 0.071465
- link link_l6: mass 0.11657 -> 0.13935
- link link_r1: mass 0.68712 -> 0.70739
- link link_r4: mass 0.080572 -> 0.087098
- link link_r6: mass 0.11657 -> 0.13935
Joints:
- added joint joint_head_pan: type revolute, parent base_link, child link_head_pan, origin xyz=0.05 0 1.429 rpy=-3.1416 0 0, axis 0 0 1, limit lower=-1.57 upper=1.57 effort=0 velocity=0
- added joint joint_head_tilt: type revolute, parent link_head_pan, child link_head_tilt, origin xyz=0 0 0 rpy=1.5708 0 0, axis 0 0 1, limit lower=-3.14 upper=3.14 effort=0 velocity=0
- joint joint_l1: limit lower=0 upper=1 effort=0 velocity=0 -> lower=0 upper=1.2 effort=0 velocity=0; origin xyz=-0.025 0.0755 0.2178 rpy=0 0 1.5708 -> xyz=-0.0405 0.065 0.227 rpy=0 0 1.5708
- joint joint_l2: origin xyz=0.075 0 0 rpy=0 0 -0.18555 -> xyz=0.068 0 0 rpy=0 0 -0.18555
- joint joint_l4: limit lower=-1.57 upper=1.57 effort=0 velocity=0 -> lower=-3.14 upper=3.14 effort=0 velocity=0; origin xyz=0.265 0 -0.079 rpy=3.1416 0 0 -> xyz=0.265 0 -0.087 rpy=3.1416 0 0
- joint joint_l6: origin xyz=0 0 0 rpy=1.5708 0 0 -> xyz=0 0 0 rpy=-1.5708 0 0
- joint joint_l7l: origin xyz=0.063 0 0.195 rpy=1.5708 -1.5708 0 -> xyz=0.078 0 0.195 rpy=1.5708 -1.5708 0
- joint joint_l7r: origin xyz=0.063 0 0.195 rpy=1.5708 -1.5708 0 -> xyz=0.078 0 0.195 rpy=1.5708 -1.5708 0
- joint joint_r1: limit lower=0 upper=1 effort=0 velocity=0 -> lower=0 upper=1.2 effort=0 velocity=0; origin xyz=-0.025 -0.0755 0.2178 rpy=0 0 -1.5708 -> xyz=-0.0405 -0.065 0.227 rpy=0 0 -1.5708
- joint joint_r2: origin xyz=0.075 0 0 rpy=0 0 0.18555 -> xyz=0.068 0 0 rpy=0 0 0.18555
- joint joint_r4: limit lower=-1.57 upper=1.57 effort=0 velocity=0 -> lower=-3.14 upper=3.14 effort=0 velocity=0; origin xyz=0.265 0 -0.079 rpy=3.1416 0 0 -> xyz=0.265 0 -0.087 rpy=3.1416 0 0
- joint joint_r7l: origin xyz=0.063 0 0.195 rpy=1.5708 -1.5708 0 -> xyz=0.078 0 0.195 rpy=1.5708 -1.5708 0
- joint joint_r7r: origin xyz=0.063 0 0.195 rpy=1.5708 -1.5708 0 -> xyz=0.078 0 0.195 rpy=1.5708 -1.5708 0

Commit message: Fix wrong urdf export, never success once!

File: urdf/astra_description.urdf (robot description, URDF)
Before this commit: robot astra_description, 21 links, 20 joints
Joints:
- joint joint_l4: origin xyz=0.265 0 -0.087 rpy=3.1416 0 0 -> xyz=0.265 0 -0.087 rpy=3.1416 0 3.1416

File: urdf/astra_description_rel.urdf (robot description, URDF)
Before this commit: robot astra_description, 21 links, 20 joints
Joints:
- joint joint_l4: origin xyz=0.265 0 -0.087 rpy=3.1416 0 0 -> xyz=0.265 0 -0.087 rpy=3.1416 0 3.1416

Commit message: Move eef to ball joint for better z-axis stablity (if we set eef to the gripper tip, the gripper pos change will cause z-axis move, which will cause whole system unstable TODO add velocity control)

File: urdf/astra_description.urdf (robot description, URDF)
Before this commit: robot astra_description, 21 links, 20 joints
Links:
- added link link_lee_teleop, mass 0.0; collision cylinder length=0.0 radius=0.0
- added link link_ree_teleop, mass 0.0; collision cylinder length=0.0 radius=0.0
Joints:
- added joint joint_lee_teleop: type fixed, parent link_l6, child link_lee_teleop, origin xyz=0 0 0 rpy=0 -1.5708 0, axis 0 0 0
- added joint joint_ree_teleop: type fixed, parent link_r6, child link_ree_teleop, origin xyz=0 0 0 rpy=0 -1.5708 0

File: urdf/astra_description_rel.urdf (robot description, URDF)
Before this commit: robot astra_description, 21 links, 20 joints
Links:
- added link link_lee_teleop, mass 0.0; collision cylinder length=0.0 radius=0.0
- added link link_ree_teleop, mass 0.0; collision cylinder length=0.0 radius=0.0
Joints:
- added joint joint_lee_teleop: type fixed, parent link_l6, child link_lee_teleop, origin xyz=0 0 0 rpy=0 -1.5708 0, axis 0 0 0
- added joint joint_ree_teleop: type fixed, parent link_r6, child link_ree_teleop, origin xyz=0 0 0 rpy=0 -1.5708 0

Commit message: Add eef support

File: urdf/astra_description.urdf (robot description, URDF)
Before this commit: robot astra_description, 23 links, 22 joints
Joints:
- joint joint_lee_teleop: origin xyz=0 0 0 rpy=0 -1.5708 0 -> xyz=0.020 0.0 0.195 rpy=0 -1.5708 0
- joint joint_ree_teleop: origin xyz=0 0 0 rpy=0 -1.5708 0 -> xyz=0.020 0.0 0.195 rpy=0 -1.5708 0

File: urdf/astra_description_rel.urdf (robot description, URDF)
Before this commit: robot astra_description, 23 links, 22 joints
Joints:
- joint joint_lee_teleop: origin xyz=0 0 0 rpy=0 -1.5708 0 -> xyz=0.020 0.0 0.195 rpy=0 -1.5708 0
- joint joint_ree_teleop: origin xyz=0 0 0 rpy=0 -1.5708 0 -> xyz=0.020 0.0 0.195 rpy=0 -1.5708 0

Commit message: Add different teleop tag

File: urdf/astra_description.urdf (robot description, URDF)
Before this commit: robot astra_description, 23 links, 22 joints
Joints:
- joint joint_lee_teleop: origin xyz=0.020 0.0 0.195 rpy=0 -1.5708 0 -> xyz=0.020 0.0 0.200 rpy=0 -1.5708 0
- joint joint_ree_teleop: origin xyz=0.020 0.0 0.195 rpy=0 -1.5708 0 -> xyz=0.020 0.0 0.200 rpy=0 -1.5708 0
